File: RAMEXPB_V3.kicad_pcb (KiCad board)
At the start: 2 copper layers, 137 x 92 mm, 74 parts, among them J10 (RP3), J11 JST_06, J12 JST_06, J4 (U12E), J5 (U13E), J8 (U4F), J9 (RP2), U1 74HCT32, U10 74HCT253, U11 74HCT253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

Commit message: 74139 outputs fixed
Connections:
- R5 pad 1: Net-(U3A-~{Q1}) -> Net-(U3A-~{Q2})
- R7 pad 1: Net-(U3B-~{Q1}) -> Net-(U3B-~{Q2})
- U3 pad 10: unconnected-(U3B-~{Q2}-Pad10) -> Net-(U3B-~{Q2})
- U3 pad 11: Net-(U3B-~{Q1}) -> unconnected-(U3B-~{Q1}-Pad11)
- U3 pad 5: Net-(U3A-~{Q1}) -> unconnected-(U3A-~{Q1}-Pad5)
- U3 pad 6: unconnected-(U3A-~{Q2}-Pad6) -> Net-(U3A-~{Q2})
Routing:
- net Net-(U3B-~{Q2}): track 0.00 -> 14.7 mm
- net Net-(U3B-~{Q1}): track 14.7 -> 0.00 mm
- net Net-(U3A-~{Q1}): track 8.88 -> 0.00 mm
- net Net-(U3A-~{Q2}): track 0.00 -> 8.35 mm
Other:
- board text added: "V1.3"
- board text removed: "V1.2"
